File: Scale/scale_200/_autosave-scale_200.kicad_sch (KiCad schematic)
At the start: 39 parts, among them J1 Conn_ARM_JTAG_SWD_10, J2 Conn_01x06_Socket, J3 12V PSU, J4 Conn_01x03_Socket, J5 Conn_01x06_Socket, U1 STM32F103C8Tx, U2 W25Q32JVSS, U3 MC33063AD

Commit message: scale done. Just GERBER left
Parts:
- J3: footprint Connector_PinSocket_2.54mm:PinSocket_1x02_P2.54mm_Horizontal -> Connector_PinSocket_2.54mm:PinSocket_1x02_P2.54mm_Vertical
Changed lines of the file:
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@@
 			)
 		)
-		(property "Footprint" "Connector_PinSocket_2.54mm:PinSocket_1x02_P2.54mm_Horizontal"
+		(property "Footprint" "Connector_PinSocket_2.54mm:PinSocket_1x02_P2.54mm_Vertical"
 			(at 36.83 123.19 0)
 			(effects
