File: Box/bottom/box_bottom/box_bottom.kicad_pcb (KiCad board)
At the start: 2 copper layers, 75 x 75 mm, 70 parts, among them Q1 1N7002, Q2 1N7002, Q3 NTS4173, Q4 NTS4173, SW1 BUTTON1, U1 SN74LVC2T45, U2 SN74LVC2T45, U3 SN74LVC2T45, U4 SN74LVC2T45, U5 ESDA5V3SC6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

Commit message: first commit, local repository
Parts:
- moved G*** 3.00 mm to (215.2, 78.2)
Routing:
- added copper zone on F.Cu, net (none)
