File: Box/box_side/box_side.kicad_sch (KiCad schematic)
At the start: 64 parts, among them SW1 BUTTON1, SW2 BUTTON1, U1 STM32H742Vx, U2 LM1117, U3 LD39050PU, X1 CONN-02P1LA, X10 ST-MORPHO-CN10, X2 CONN-02P1LA, X3 CONN-02P1L, X4 ST-MORPHO-CN7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

Commit message: first commit, local repository
Parts:
- removed D1: 0603G, OPTOEL:LED-0603, symbol nuco-v-rescue:LED-COMMON
- removed D2: 0603R, OPTOEL:LED-0603, symbol nuco-v-rescue:LED-COMMON
- removed SB11, SB12, SB13, SB14: JUMPER, SMD-CMN:SMD-0603R, symbol nuco-v-rescue:JUMPER-COMMON
- added D1, D2: LED, LED_SMD:LED_0805_2012Metric_Pad1.15x1.40mm_HandSolder, symbol Device:LED
- C1, C11, C13, C14, C15, C16, C17, C18, C19, C2, C20, C21, C3, C4, C5, C6, C7, C9: footprint SMD-CMN:SMD-0603C -> Capacitor_SMD:C_0603_1608Metric_Pad1.08x0.95mm_HandSolder
- C10: footprint SMD-CMN:SMD-0805C -> Capacitor_SMD:C_0603_1608Metric_Pad1.08x0.95mm_HandSolder
- C12, C8: footprint SMD-CMN:SMD-1206C -> Capacitor_SMD:C_0805_2012Metric_Pad1.18x1.45mm_HandSolder
- D3: footprint SMD-SOT:SOD-123F -> Diode_SMD:D_SOD-123F
- L1: footprint SMD-CMN:SMD-0603L -> Inductor_SMD:L_0805_2012Metric_Pad1.05x1.20mm_HandSolder
- R1, R2, R3, R4, R5, R6, R7, R8, R9, SB1, SB10, SB15, SB16, SB17, SB6, SB7, SB8, SB9: footprint SMD-CMN:SMD-0603R -> Resistor_SMD:R_0603_1608Metric_Pad0.98x0.95mm_HandSolder
- SW1, SW2: footprint SWITCHES:B3U-1000P-B -> Button_Switch_SMD:SW_SPST_PTS645
- U1: footprint SMD-QFN:QFPX50P140X140-100 -> Package_QFP:LQFP-100_14x14mm_P0.5mm
- U2: footprint SMD-SOT:SOT-223-3 -> Package_TO_SOT_SMD:SOT-223
- U3: footprint SMD-QFN:DFNX95P030X030-6 -> Package_DFN_QFN:DFN-6-1EP_2x1.8mm_P0.5mm_EP1.2x1.6mm
- X1, X2, X3: footprint CONNFLY:DS1021-1X02S61 -> Connector_PinSocket_2.54mm:PinSocket_1x02_P2.54mm_Vertical
- X10, X4: footprint CONNFLY:DS1021-2X19S61 -> Connector_PinSocket_1.27mm:PinSocket_2x19_P1.27mm_Vertical_SMD
- X5: footprint CONNFLY:DS1023-1X08A -> Connector_PinSocket_2.54mm:PinSocket_1x08_P2.54mm_Vertical
- X6: footprint CONNFLY:DS1025-1X06S61 -> Connector_PinSocket_2.54mm:PinSocket_1x06_P2.54mm_Vertical
- X7: footprint CONNFLY:DS1021-1X03S61 -> Connector_PinSocket_2.54mm:PinSocket_1x03_P2.54mm_Vertical
- X8: footprint CONNFLY:DS1023-1X10A -> Connector_PinSocket_2.54mm:PinSocket_2x05_P2.54mm_Vertical
- X9: footprint CONNFLY:DS1021-2X04S61 -> Connector_PinSocket_2.54mm:PinSocket_1x08_P2.54mm_Vertical
- Y1: footprint QUARTZ:KX-327L -> Crystal:Crystal_SMD_EuroQuartz_EQ161-2Pin_3.2x1.5mm_HandSoldering
- Y2: footprint QUARTZ:KX-3H -> Crystal:Crystal_SMD_5032-2Pin_5.0x3.2mm
Connections:
- net PA0: no longer X4.28 (PA0)
- net PA1: no longer X4.30 (PA1)
- net PA10: no longer X10.33 (PA10)
- net PA11: no longer X10.14 (PA11)
- net PA12: now also X4.9; no longer X10.12 (PA12)
- net PA13: no longer X4.13 (PA13)
- net PA14: now also X4.10; no longer X4.15 (PA14)
- net PA15: now also X4.11; no longer X4.17 (PA15)
- net PA2: now also X10.19 (PC7); no longer X10.35 (PA2)
- net PA3: now also X10.18; no longer X10.37 (PA3)
- net PA4: no longer X4.32 (PA4)
- net PA5: now also X10.17 (PB6); no longer X10.11 (PA5)
- net PA6: now also X10.16 (PB12); no longer X10.13 (PA6)
- net PA8: no longer X10.23 (PA8)
- net PA9: no longer X10.21 (PA9)
- net PB0: no longer X4.34 (PB0)
- net PB1: now also X10.12 (PA12); no longer X10.24 (PB1)
- net PB10: now also X10.10; no longer X10.25 (PB10)
- net PB11: no longer X10.18
- net PB12: now also X10.4 (PC6); no longer X10.16 (PB12)
- net PB13: now also X10.3 (PB8), X8.1; no longer X10.30 (PB13)
- net PB14: now also X10.2 (PC8); no longer X10.28 (PB14)
- net PB15: now also X10.1 (PC9); no longer X10.26 (PB15)
- net PB2: now also X10.11 (PA5); no longer X10.22 (PB2)
- net PB3: now also X4.23 (PC13), X4.31 (PH1); no longer X10.31 (PB3)
- net PB4: no longer X10.27 (PB4)
- net PB5: now also X4.25 (PC14); no longer X10.29 (PB5)
- net PB6: now also X4.26; no longer X10.17 (PB6)
- net PB7: now also X4.27 (PC15); no longer X4.21 (PB7)
- net PB8: now also X4.28 (PA0); no longer X10.3 (PB8), X8.1
- net PB9: now also X4.29 (PH0); no longer X10.5 (PB9), X8.2
- net PC0: now also X10.24 (PB1); no longer X4.38 (PC0/PB8)
- net PC1: now also X10.23 (PA8); no longer X4.36 (PC1/PB9)
- net PC10: no longer X4.1 (PC10)
- net PC11: now also X4.13 (PA13); no longer X4.2 (PC11)
- net PC12: now also X4.14 (RESET), X5.3; no longer X4.3 (PC12)
- net PC13: no longer X4.23 (PC13)
- net PC2: now also X10.22 (PB2)
- net PC3: now also X10.21 (PA9)
- net PC4: now also X10.14 (PA11); no longer X10.34 (PC4)
- net PC5: now also X10.13 (PA6)
- net PC6: now also X4.1 (PC10); no longer X10.4 (PC6)
- net PC7: now also X4.2 (PC11); no longer X10.19 (PC7)
- net PC8: now also X4.3 (PC12); no longer X10.2 (PC8)
- net PC9: now also X4.4 (PD2); no longer X10.1 (PC9)
- net PD0: now also X4.15 (PA14); no longer X4.9
- net PD1: no longer X4.11
- net PD2: now also X4.17 (PA15); no longer X4.4 (PD2)
- net PD3: no longer X4.10
- net PD4: no longer X4.26
- net PD5: no longer X10.10
- net PD6: now also X4.21 (PB7); no longer X10.36
- net PD7: no longer X10.38
- net PGND: now also X4.30 (PA1), X4.32 (PA4), X4.34 (PB0), X4.36 (PC1/PB9), X4.38 (PC0/PB8)
- net VDD: now also D2.2 (A)
- net nRST: no longer X4.14 (RESET), X5.3
- net at R2.1 (R1): now also D2.1 (K)
- net at SB1.1 (J1): now also D1.2 (A)
- net at R1.1 (R1): now also D1.1 (K)
- new net: X10.5 (PB9), X8.2
Other:
- moved on the sheet: X6, X9
