File: Box/box_side/box_side_red.kicad_pcb (KiCad board)
At the start: 2 copper layers, 75 x 101.5 mm, 67 parts, among them SW1 BUTTON1, SW2 BUTTON1, U1 STM32H742Vx, U2 LM1117, U3 LD39050PU, X1 CONN-02P1LA, X10 ST-MORPHO-CN10, X2 CONN-02P1LA, X3 CONN-02P1L, X4 ST-MORPHO-CN7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

Commit message: all gerbers done
Routing:
- net PGND: track 89.6 -> 90.7 mm, vias 34 -> 33
Other:
- board text added: "{dblquote}Практические навыки работы инженера-радиоэлектронщика{dblquote}"
- board text added: "Выпускнику курса"
- board text added: "С ОТЛИЧИЕМ!"
